File: Blackbox.kicad_pcb (KiCad board)
At the start: 4 copper layers, 77 x 34.5 mm, 43 parts, among them CN1 SM04B-SRSS-TB (LF)(SN), U1 SN65HVD232DR, U2 STM32G0B1CCT6, U3 BM06B-SRSS-TB(LF)(SN), X2 DSX321G-48M

Commit message: Final Version of the BlackBox PCB
Parts:
- added G***: LOGO, LOGO, F.Cu at (145.0, 118.0)

Commit message: BlackBox PCB For Freyja Rocket
Parts:
- added G***: LOGO, LOGO, F.Cu at (161.5, 89.0)
- moved REF** 2.55 mm to (176.0, 89.5)
- moved REF** 2.50 mm to (176.0, 117.5)
- moved REF** 1.80 mm to (106.0, 89.5)
- moved REF** 1.58 mm to (106.0, 117.5)
Routing:
- net CLK: track 24.8 -> 27.1 mm
- net GND: track 48.0 -> 49.0 mm
- net VDD: track 40.6 -> 41.2 mm
Other:
- board size 77 x 34.5 mm -> 77 x 35 mm
